File: KiCAD Projects/skogaslider-main-pcb/skogaslider-main-pcb.kicad_pcb (KiCad board)
At the start: 2 copper layers, 541 x 152.4 mm, 30 parts, among them J1 Conn_01x02, J2 USB_B_Micro, U1 W25Q128JVS, U2 NCP1117-3.3_SOT223, U3 RP2040, U4 MPR121QR2, Y1 ABLS-12.000MHZ-B4-T

Commit message: Almost final schematic for the main slider, minus a couple of small tweaks. Significant progress on slider board layout. MPR121 layouts are essentially complete minus the key wiring. USB C ports and LEDs are also laid out.
Parts:
- removed Touch Slider: Conn_02x16_Top_Bottom, Chunithm_Touch_Pad:Pads
- added C18: 0.1u, Capacitor_SMD:C_0402_1005Metric, F.Cu at (321.4, 304.4)
- added C19: 0.1u, Capacitor_SMD:C_0402_1005Metric, F.Cu at (437.4, 304.4)
- added C20: 100n, Capacitor_SMD:C_0402_1005Metric, F.Cu at (394.1, 394.5)
- added C21: 0.1u, Capacitor_SMD:C_0402_1005Metric, F.Cu at (548.5, 302.7)
- added C22: 0.1u, Capacitor_SMD:C_0402_1005Metric, F.Cu at (553.4, 304.4)
- added C23: 27p, Capacitor_SMD:C_0402_1005Metric, F.Cu at (379.3, 378.2)
- added C24: 27p, Capacitor_SMD:C_0402_1005Metric, F.Cu at (383.2, 378.5)
- added C25: 100nF, Capacitor_SMD:C_0402_1005Metric, F.Cu at (218.3, 291.6)
- added C26: 100nF, Capacitor_SMD:C_0402_1005Metric, F.Cu at (228.0, 291.6)
- added C27: 100nF, Capacitor_SMD:C_0402_1005Metric, F.Cu at (237.7, 291.6)
- added C28: 100nF, Capacitor_SMD:C_0402_1005Metric, F.Cu at (247.3, 291.6)
- added C29: 100nF, Capacitor_SMD:C_0402_1005Metric, F.Cu at (257.0, 291.6)
- added C30: 100nF, Capacitor_SMD:C_0402_1005Metric, F.Cu at (266.7, 291.6)
- added C31: 100nF, Capacitor_SMD:C_0402_1005Metric, F.Cu at (276.3, 291.6)
- added C32: 100nF, Capacitor_SMD:C_0402_1005Metric, F.Cu at (286.0, 291.6)
- added C33: 100nF, Capacitor_SMD:C_0402_1005Metric, F.Cu at (295.7, 291.6)
- added C34: 100nF, Capacitor_SMD:C_0402_1005Metric, F.Cu at (305.3, 291.6)
- added C35: 100nF, Capacitor_SMD:C_0402_1005Metric, F.Cu at (315.0, 291.6)
- added C36: 100nF, Capacitor_SMD:C_0402_1005Metric, F.Cu at (324.7, 291.6)
- added C37: 100nF, Capacitor_SMD:C_0402_1005Metric, F.Cu at (334.3, 291.6)
- added C38: 100nF, Capacitor_SMD:C_0402_1005Metric, F.Cu at (344.0, 291.6)
- added C39: 100nF, Capacitor_SMD:C_0402_1005Metric, F.Cu at (353.7, 291.6)
- added C40: 100nF, Capacitor_SMD:C_0402_1005Metric, F.Cu at (363.3, 291.6)
- added C41: 100nF, Capacitor_SMD:C_0402_1005Metric, F.Cu at (373.0, 291.6)
- added C42: 100nF, Capacitor_SMD:C_0402_1005Metric, F.Cu at (382.7, 291.6)
- added C43: 100nF, Capacitor_SMD:C_0402_1005Metric, F.Cu at (392.3, 291.6)
- added C44: 100nF, Capacitor_SMD:C_0402_1005Metric, F.Cu at (402.0, 291.6)
- added C45: 100nF, Capacitor_SMD:C_0402_1005Metric, F.Cu at (411.7, 291.6)
- added C46: 100nF, Capacitor_SMD:C_0402_1005Metric, F.Cu at (421.3, 291.6)
- added C47: 100nF, Capacitor_SMD:C_0402_1005Metric, F.Cu at (431.0, 291.6)
- added C48: 100nF, Capacitor_SMD:C_0402_1005Metric, F.Cu at (440.7, 291.6)
- added C49: 100nF, Capacitor_SMD:C_0402_1005Metric, F.Cu at (450.3, 291.6)
- added C50: 100nF, Capacitor_SMD:C_0402_1005Metric, F.Cu at (460.0, 291.6)
- added C51: 100nF, Capacitor_SMD:C_0402_1005Metric, F.Cu at (469.7, 291.6)
- added C52: 100nF, Capacitor_SMD:C_0402_1005Metric, F.Cu at (479.3, 291.6)
- added C53: 100nF, Capacitor_SMD:C_0402_1005Metric, F.Cu at (489.0, 291.6)
- added C54: 100nF, Capacitor_SMD:C_0402_1005Metric, F.Cu at (498.7, 291.6)
- added C55: 100nF, Capacitor_SMD:C_0402_1005Metric, F.Cu at (508.3, 291.6)
- added C56: 100nF, Capacitor_SMD:C_0402_1005Metric, F.Cu at (518.0, 291.6)
- added C57: 100nF, Capacitor_SMD:C_0603_1608Metric, F.Cu at (468.2, 425.3)
- added C58: 100nF, Capacitor_SMD:C_0402_1005Metric, F.Cu at (527.7, 291.6)
- added C59: 100nF, Capacitor_SMD:C_0402_1005Metric, F.Cu at (537.3, 291.6)
- added C60: 100nF, Capacitor_SMD:C_0402_1005Metric, F.Cu at (547.0, 291.6)
- added C61: 100nF, Capacitor_SMD:C_0402_1005Metric, F.Cu at (556.7, 291.6)
- added C62: 100nF, Capacitor_SMD:C_0402_1005Metric, F.Cu at (566.3, 291.6)
- added C63: 100nF, Capacitor_SMD:C_0402_1005Metric, F.Cu at (576.0, 291.6)
- added C64: 100nF, Capacitor_SMD:C_0402_1005Metric, F.Cu at (585.7, 291.6)
- added C65: 100nF, Capacitor_SMD:C_0402_1005Metric, F.Cu at (595.3, 291.6)
- added C66: 100nF, Capacitor_SMD:C_0402_1005Metric, F.Cu at (605.0, 291.6)
- added C67: 100nF, Capacitor_SMD:C_0402_1005Metric, F.Cu at (614.7, 291.6)
- added C68: 100nF, Capacitor_SMD:C_0402_1005Metric, F.Cu at (624.3, 291.6)
- added C69: 100nF, Capacitor_SMD:C_0402_1005Metric, F.Cu at (634.0, 291.6)
- added C70: 100nF, Capacitor_SMD:C_0402_1005Metric, F.Cu at (643.7, 291.6)
- added C71: 100nF, Capacitor_SMD:C_0402_1005Metric, F.Cu at (653.3, 291.6)
- added C72: 100nF, Capacitor_SMD:C_0402_1005Metric, F.Cu at (663.0, 291.6)
- added D1: D_Schottky, Diode_SMD:D_SMA, F.Cu at (391.1, 153.6)
- added D10: WS2812B, WS2812B-4020:WS2812B-4020, F.Cu at (281.2, 291.1)
- added D11: WS2812B, WS2812B-4020:WS2812B-4020, F.Cu at (290.8, 291.1)
- added D12: WS2812B, WS2812B-4020:WS2812B-4020, F.Cu at (300.5, 291.1)
- added D13: WS2812B, WS2812B-4020:WS2812B-4020, F.Cu at (310.2, 291.1)
- added D14: WS2812B, WS2812B-4020:WS2812B-4020, F.Cu at (319.8, 291.1)
- added D15: WS2812B, WS2812B-4020:WS2812B-4020, F.Cu at (329.5, 291.1)
- added D16: WS2812B, WS2812B-4020:WS2812B-4020, F.Cu at (339.2, 291.1)
- added D17: WS2812B, WS2812B-4020:WS2812B-4020, F.Cu at (348.8, 291.1)
- added D18: WS2812B, WS2812B-4020:WS2812B-4020, F.Cu at (358.5, 291.1)
- added D19: WS2812B, WS2812B-4020:WS2812B-4020, F.Cu at (368.2, 291.1)
- added D2: D_Schottky, Diode_SMD:D_SMA, F.Cu at (413.2, 153.6)
- added D20: WS2812B, WS2812B-4020:WS2812B-4020, F.Cu at (377.8, 291.1)
- added D21: WS2812B, WS2812B-4020:WS2812B-4020, F.Cu at (387.5, 291.1)
- added D22: WS2812B, WS2812B-4020:WS2812B-4020, F.Cu at (397.2, 291.1)
- added D23: WS2812B, WS2812B-4020:WS2812B-4020, F.Cu at (406.8, 291.1)
- added D24: WS2812B, WS2812B-4020:WS2812B-4020, F.Cu at (416.5, 291.1)
- added D25: WS2812B, WS2812B-4020:WS2812B-4020, F.Cu at (426.2, 291.1)
- added D26: WS2812B, WS2812B-4020:WS2812B-4020, F.Cu at (435.8, 291.1)
- added D27: WS2812B, WS2812B-4020:WS2812B-4020, F.Cu at (445.5, 291.1)
- added D28: WS2812B, WS2812B-4020:WS2812B-4020, F.Cu at (455.2, 291.1)
- added D29: WS2812B, WS2812B-4020:WS2812B-4020, F.Cu at (464.8, 291.1)
- added D3: WS2812B, WS2812B-4020:WS2812B-4020, F.Cu at (213.5, 291.1)
- added D30: WS2812B, WS2812B-4020:WS2812B-4020, F.Cu at (474.5, 291.1)
- added D31: WS2812B, WS2812B-4020:WS2812B-4020, F.Cu at (484.2, 291.1)
- added D32: WS2812B, WS2812B-4020:WS2812B-4020, F.Cu at (493.8, 291.1)
- added D33: WS2812B, WS2812B-4020:WS2812B-4020, F.Cu at (503.5, 291.1)
- added D34: WS2812B, WS2812B-4020:WS2812B-4020, F.Cu at (513.2, 291.1)
- added D35: WS2812B, WS2812B-4020:WS2812B-4020, F.Cu at (522.8, 291.1)
- added D36: WS2812B, WS2812B-4020:WS2812B-4020, F.Cu at (532.5, 291.1)
- added D37: WS2812B, WS2812B-4020:WS2812B-4020, F.Cu at (542.2, 291.1)
- added D38: WS2812B, WS2812B-4020:WS2812B-4020, F.Cu at (551.8, 291.1)
- added D39: WS2812B, WS2812B-4020:WS2812B-4020, F.Cu at (561.5, 291.1)
- added D4: WS2812B, WS2812B-4020:WS2812B-4020, F.Cu at (223.2, 291.1)
- added D40: WS2812B, WS2812B-4020:WS2812B-4020, F.Cu at (571.2, 291.1)
- added D41: WS2812B, WS2812B-4020:WS2812B-4020, F.Cu at (580.8, 291.1)
- added D42: WS2812B, WS2812B-4020:WS2812B-4020, F.Cu at (590.5, 291.1)
- added D43: WS2812B, WS2812B-4020:WS2812B-4020, F.Cu at (600.2, 291.1)
- added D44: WS2812B, WS2812B-4020:WS2812B-4020, F.Cu at (609.8, 291.1)
- added D45: WS2812B, WS2812B-4020:WS2812B-4020, F.Cu at (619.5, 291.1)
- added D46: WS2812B, WS2812B-4020:WS2812B-4020, F.Cu at (629.2, 291.1)
- added D47: WS2812B, WS2812B-4020:WS2812B-4020, F.Cu at (638.8, 291.1)
- added D48: WS2812B, WS2812B-4020:WS2812B-4020, F.Cu at (648.5, 291.1)
- added D49: WS2812B, WS2812B-4020:WS2812B-4020, F.Cu at (658.2, 291.1)
- added D5: WS2812B, WS2812B-4020:WS2812B-4020, F.Cu at (232.8, 291.1)
- added D6: WS2812B, WS2812B-4020:WS2812B-4020, F.Cu at (242.5, 291.1)
- added D7: WS2812B, WS2812B-4020:WS2812B-4020, F.Cu at (252.2, 291.1)
- added D8: WS2812B, WS2812B-4020:WS2812B-4020, F.Cu at (261.8, 291.1)
- added D9: WS2812B, WS2812B-4020:WS2812B-4020, F.Cu at (271.5, 291.1)
- added J3: Conn_01x05, Connector_PinHeader_2.54mm:PinHeader_1x05_P2.54mm_Vertical, F.Cu at (417.8, 419.4)
- added J4: Conn_02x16_Top_Bottom, Chunithm_Touch_Pad:Pads, F.Cu at (204.1, 204.2)
- added J5: Conn_01x09, Connector_JST:JST_PH_S9B-PH-K_1x09_P2.00mm_Horizontal, F.Cu at (169.9, 303.6)
- added J6: Conn_01x09, Connector_JST:JST_PH_S9B-PH-K_1x09_P2.00mm_Horizontal, F.Cu at (701.3, 324.1)
- added J7: Conn_01x04, Connector_JST:JST_PH_S4B-PH-K_1x04_P2.00mm_Horizontal, F.Cu at (702.1, 339.1)
- added J8: Conn_01x04, Connector_JST:JST_PH_S4B-PH-K_1x04_P2.00mm_Horizontal, F.Cu at (170.5, 327.3)
- added Q1: BSS138, Package_TO_SOT_SMD:SOT-23, F.Cu at (421.9, 389.2)
- added R10: 75k, Resistor_SMD:R_0603_1608Metric, F.Cu at (438.8, 302.5)
- added R11: 27, Resistor_SMD:R_0603_1608Metric, F.Cu at (432.5, 374.3)
- added R12: 1.7k, Resistor_SMD:R_0603_1608Metric, F.Cu at (417.2, 156.4)
- added R13: 27, Resistor_SMD:R_0603_1608Metric, F.Cu at (432.8, 378.1)
- added R14: 3.3k, Resistor_SMD:R_0603_1608Metric, F.Cu at (421.7, 156.4)
- added R15: 10k, Resistor_SMD:R_0603_1608Metric, F.Cu at (426.2, 388.1)
- added R16: 10k, Resistor_SMD:R_0603_1608Metric, F.Cu at (426.4, 392.4)
- added R17: 10k, Resistor_SMD:R_0603_1608Metric, F.Cu at (384.8, 395.7)
- added R18: 10k, Resistor_SMD:R_0603_1608Metric, F.Cu at (550.1, 306.5)
- added R19: 10k, Resistor_SMD:R_0603_1608Metric, F.Cu at (550.1, 304.4)
- added R20: 1k, Resistor_SMD:R_0402_1005Metric, F.Cu at (389.5, 395.5)
- added R21: 50k, Resistor_SMD:R_0603_1608Metric, F.Cu at (439.0, 374.7)
- added R22: 75k, Resistor_SMD:R_0603_1608Metric, F.Cu at (554.8, 302.5)
- added R23: 1k, Resistor_SMD:R_0402_1005Metric, F.Cu at (387.0, 377.7)
- added R24: 10k, Resistor_SMD:R_0603_1608Metric, F.Cu at (463.6, 425.3)
- added R6: 5.1k, Resistor_SMD:R_0603_1608Metric, F.Cu at (394.2, 152.6)
- added R7: 5.1k, Resistor_SMD:R_0603_1608Metric, F.Cu at (419.9, 151.9)
- added R8: 5.1k, Resistor_SMD:R_0603_1608Metric, F.Cu at (416.9, 152.0)
- added R9: 75k, Resistor_SMD:R_0603_1608Metric, F.Cu at (322.8, 302.5)
- added SW1: SW_Push, TS-1187A-B-A-B:SW_TS-1187A-B-A-B, F.Cu at (356.6, 395.6)
- added SW2: SW_Push, TS-1187A-B-A-B:SW_TS-1187A-B-A-B, F.Cu at (260.2, 167.2)
- added SW3: SW_Push, TS-1187A-B-A-B:SW_TS-1187A-B-A-B, F.Cu at (273.8, 166.9)
- added SW4: SW_Push, TS-1187A-B-A-B:SW_TS-1187A-B-A-B, F.Cu at (289.1, 167.4)
- added TP1: TestPoint, TestPoint:TestPoint_Pad_D1.5mm, F.Cu at (383.1, 126.0)
- added TP2: TestPoint, TestPoint:TestPoint_Pad_D1.5mm, F.Cu at (390.7, 126.0)
- added TP3: TestPoint, TestPoint:TestPoint_Pad_D1.5mm, F.Cu at (398.3, 126.0)
- added TP4: TestPoint, TestPoint:TestPoint_Pad_D1.5mm, F.Cu at (405.9, 126.0)
- added U5: RP2040, RP2040_minimal:RP2040-QFN-56, F.Cu at (423.5, 374.1)
- added U6: M24C02-RMN, Package_SO:SOIC-8_3.9x4.9mm_P1.27mm, F.Cu at (470.0, 389.1)
- added U7: W25Q128JVS, Package_SO:SOIC-8_5.23x5.23mm_P1.27mm, F.Cu at (390.1, 401.2)
- added U8: MPR121QR2, Package_DFN_QFN:UQFN-20_3x3mm_P0.4mm, F.Cu at (551.8, 300.7)
- added U9: 74HC4051, Package_SO:TSSOP-16_4.4x5mm_P0.65mm, F.Cu at (466.0, 417.5)
- C1, C2: value 27p -> 100n
- C10, C8: value 1u -> 100n
- C11, C12, C17: value 100n -> 0.1u
- C13: value 100n -> 22u; footprint Capacitor_SMD:C_0402_1005Metric -> Capacitor_SMD:C_0805_2012Metric
- C14: value 10u -> 22u
- C15, C16: value 100n -> 1u
- C5: value 10u -> 100n; footprint Capacitor_SMD:C_0805_2012Metric -> Capacitor_SMD:C_0402_1005Metric
- J1: value Conn_01x02 -> USB_C_Receptacle_USB2.0; footprint Connector_PinHeader_2.54mm:PinHeader_1x02_P2.54mm_Vertical -> Connector_USB:USB_C_Receptacle_HRO_TYPE-C-31-M-12
- J2: value USB_B_Micro -> USB_C_Receptacle_USB2.0; footprint RP2040_minimal:USB_Micro-B_Amphenol_10103594-0001LF_Horizontal_modified -> Connector_USB:USB_C_Receptacle_HRO_TYPE-C-31-M-12
- R1, R3: value 1k -> 10k; footprint Capacitor_SMD:C_0402_1005Metric -> Resistor_SMD:R_0603_1608Metric
- R2: value DNF -> 10k; footprint Capacitor_SMD:C_0402_1005Metric -> Resistor_SMD:R_0603_1608Metric
- R4: value 27 -> 10k; footprint Capacitor_SMD:C_0402_1005Metric -> Resistor_SMD:R_0603_1608Metric
- R5: value 27 -> 5.1k; footprint Capacitor_SMD:C_0402_1005Metric -> Resistor_SMD:R_0603_1608Metric
- U1: value W25Q128JVS -> AMS1117-3.3; footprint Package_SO:SOIC-8_5.23x5.23mm_P1.27mm -> Package_TO_SOT_SMD:SOT-223-3_TabPin2
- U2: value NCP1117-3.3_SOT223 -> MPR121QR2; footprint Package_TO_SOT_SMD:SOT-223-3_TabPin2 -> Package_DFN_QFN:UQFN-20_3x3mm_P0.4mm
- U3: value RP2040 -> MPR121QR2; footprint RP2040_minimal:RP2040-QFN-56 -> Package_DFN_QFN:UQFN-20_3x3mm_P0.4mm
- U4: value MPR121QR2 -> USBLC6-2P6; footprint Package_DFN_QFN:UQFN-20_3x3mm_P0.4mm -> Package_TO_SOT_SMD:SOT-666
- moved J1 275.5 mm to (418.6, 144.7), turned to 180 degrees
- moved J2 250.7 mm to (396.5, 144.7), turned to 180 degrees
- moved R5 242.4 mm to (398.8, 152.6), turned to -90 degrees
- moved C14 240.5 mm to (400.8, 159.3), turned to 90 degrees
- moved C13 234.3 mm to (410.8, 159.3), turned to 90 degrees
- moved C17 221.5 mm to (395.3, 156.1)
- moved C3 219.2 mm to (425.0, 361.8)
- moved R3 216.5 mm to (434.1, 306.5)
- moved C5 214.9 mm to (433.6, 361.4)
- moved U4 210.9 mm to (396.5, 152.6), turned to -90 degrees
- moved C10 207.9 mm to (433.4, 366.0)
- moved C2 206.8 mm to (420.6, 361.4)
- moved C15 206.2 mm to (439.9, 359.5)
- moved C7 202.3 mm to (420.4, 366.0)
- moved C4 196.3 mm to (429.2, 361.4)
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Connections:
- C1 pad 1: /XIN -> +1V1
- C11 pad 1: +3V3 -> GND
- C11 pad 2: GND -> +3V3
- C12 pad 1: +3V3 -> GND
- C12 pad 2: GND -> +3V3
- C13 pad 1: +3V3 -> +5V
- C15 pad 1: +3V3 -> +1V1
- C17 pad 1: +3V3 -> GND
- C17 pad 2: GND -> +5V
- C2 pad 1: Net-(C2-Pad1) -> +1V1
- C3 pad 1: VBUS -> +3V3
- C6 pad 1: +1V1 -> +3V3
- C7 pad 1: +1V1 -> +3V3
- C8 pad 1: +1V1 -> +3V3
- R1 pad 1: /QSPI_SS -> +3V3
- R1 pad 2: /~{USB_BOOT} -> /SCL
- R2 pad 2: /QSPI_SS -> /SDA
- R3 pad 1: /XOUT -> +3V3
- R3 pad 2: Net-(C2-Pad1) -> /SCL
- R4 pad 1: /USB_D+ -> +3V3
- R4 pad 2: Net-(R4-Pad2) -> /SDA
- R5 pad 1: /USB_D- -> Net-(J2-PadA5)
- R5 pad 2: Net-(R5-Pad2) -> GND
- U1 pad 1: /QSPI_SS -> GND
- U1 pad 2: /QSPI_SD1 -> +3V3
- U1 pad 3: /QSPI_SD2 -> +5V
- U2 pad 1: GND -> unconnected-(U2-Pad1)
- U2 pad 2: +3V3 -> /SCL
- U2 pad 3: VBUS -> /SDA
- U3 pad 1: +3V3 -> unconnected-(U3-Pad1)
- U3 pad 10: +3V3 -> /KEY_22
- U3 pad 11: /GPIO8 -> /KEY_21
- U3 pad 12: /GPIO9 -> /KEY_20
- U3 pad 13: /GPIO10 -> /KEY_19
- U3 pad 14: /GPIO11 -> /KEY_18
- U3 pad 15: /GPIO12 -> /KEY_17
- U3 pad 16: /GPIO13 -> /KEY_16
- U3 pad 17: /GPIO14 -> /KEY_15
- U3 pad 18: /GPIO15 -> /KEY_14
- U3 pad 19: GND -> /KEY_13
- U3 pad 2: /GPIO0 -> /SCL
- U3 pad 20: /XIN -> +3V3
- U3 pad 3: /GPIO1 -> /SDA
- U3 pad 4: /GPIO2 -> /SDA
- U3 pad 5: /GPIO3 -> Net-(C19-Pad2)
- U3 pad 6: /GPIO4 -> GND
- U3 pad 7: /GPIO5 -> Net-(R10-Pad2)
- U3 pad 8: /GPIO6 -> /KEY_24
- U3 pad 9: /GPIO7 -> /KEY_23
- U4 pad 1: unconnected-(U4-Pad1) -> /PRE_USB_D-
- U4 pad 2: unconnected-(U4-Pad2) -> GND
- U4 pad 3: unconnected-(U4-Pad3) -> /PRE_USB_D+
- U4 pad 4: unconnected-(U4-Pad4) -> /USB_D-
- U4 pad 5: unconnected-(U4-Pad5) -> +5V
- U4 pad 6: unconnected-(U4-Pad6) -> /USB_D+
- Y1 pad 2: Net-(C2-Pad1) -> Net-(C24-Pad1)
Routing:
- net +5V: track 0.00 -> 714.6 mm, vias 0 -> 1
- net GND: track 0.00 -> 99.9 mm, vias 0 -> 2
- net +3V3: track 0.00 -> 34.6 mm
- net /SCL: track 0.00 -> 17.8 mm
- net Net-(D1-Pad2): track 0.00 -> 16.6 mm
- net Net-(J1-PadA4): track 0.00 -> 16.6 mm
- net Net-(D37-Pad2): track 0.00 -> 14.7 mm
- net Net-(D17-Pad2): track 0.00 -> 14.7 mm
- net Net-(D43-Pad2): track 0.00 -> 14.7 mm
- net Net-(D29-Pad2): track 0.00 -> 14.7 mm
- net Net-(D23-Pad2): track 0.00 -> 14.7 mm
- net Net-(D25-Pad2): track 0.00 -> 14.7 mm
- net Net-(D27-Pad2): track 0.00 -> 14.7 mm
- net Net-(D21-Pad2): track 0.00 -> 14.7 mm
- net Net-(D3-Pad2): track 0.00 -> 14.7 mm
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- added copper zone on F.Cu, net GND
Other:
- board outline removed

Commit message: More layout progress for the main slider PCB
Parts:
- C13, C14: footprint Capacitor_SMD:C_0805_2012Metric -> Capacitor_Tantalum_SMD:CP_EIA-1608-08_AVX-J
- moved SW1 108.6 mm to (457.9, 356.8)
- moved SW3 84.3 mm to (354.3, 142.2)
- moved SW4 84.3 mm to (369.7, 142.7)
- moved SW2 84.3 mm to (340.7, 142.5)
- moved R17 59.5 mm to (439.4, 372.1)
- moved R20 59.5 mm to (444.1, 371.9)
- moved U7 59.5 mm to (444.7, 377.6)
- moved C20 59.5 mm to (448.7, 370.9)
- moved R21 33.3 mm to (408.6, 388.4)
- moved Y1 17.8 mm to (402.9, 371.3)
- moved C23 17.8 mm to (397.1, 378.5)
- moved C24 17.8 mm to (401.1, 378.9)
- moved R23 17.8 mm to (404.8, 378.0)
- moved R12 7.41 mm to (423.1, 151.9), turned to -90 degrees
- moved R11 7.14 mm to (434.4, 381.2)
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Connections:
- D2 pad 2: Net-(J1-PadA4) -> Net-(D2-Pad2)
- J1 pad A4: Net-(J1-PadA4) -> Net-(D2-Pad2)
- J1 pad A9: Net-(J1-PadA4) -> Net-(D2-Pad2)
- J1 pad B4: Net-(J1-PadA4) -> Net-(D2-Pad2)
- J1 pad B9: Net-(J1-PadA4) -> Net-(D2-Pad2)
- R12 pad 1: +5V -> Net-(D2-Pad2)
Routing:
- net Net-(D2-Pad2): track 0.00 -> 25.6 mm
- net Net-(J1-PadA4): track 16.6 -> 0.00 mm
- net +5V: track 714.6 -> 711.2 mm
- net GND: track 99.9 -> 97.7 mm
- removed copper zone on F.Cu, net GND

Commit message: PCB layout is almost complete for the mainboard, minus the board cuts, mounting holes, and power/ground planes
Parts:
- removed J7, J8: Conn_01x04, Connector_JST:JST_PH_S4B-PH-K_1x04_P2.00mm_Horizontal
- added C73: 100n, Capacitor_SMD:C_0201_0603Metric, F.Cu at (356.1, 304.7)
- C1, C10, C15, C16, C2, C4, C5, C6, C7, C8, C9: footprint Capacitor_SMD:C_0402_1005Metric -> Capacitor_SMD:C_0201_0603Metric
- C3: value 10u -> 100n; footprint Capacitor_SMD:C_0805_2012Metric -> Capacitor_SMD:C_0201_0603Metric
- J3: value Conn_01x05 -> Conn_01x03; footprint Connector_PinHeader_2.54mm:PinHeader_1x05_P2.54mm_Vertical -> Connector_PinHeader_2.54mm:PinHeader_1x03_P2.54mm_Vertical
- J5, J6: value Conn_01x09 -> HDMI_A_No_Video; footprint Connector_JST:JST_PH_S9B-PH-K_1x09_P2.00mm_Horizontal -> Skogaslider_Custom_Footprints:HDMI_Connector_SMD
- R20: footprint Resistor_SMD:R_0402_1005Metric -> Resistor_SMD:R_0603_1608Metric
- moved SW3 180.3 mm to (527.2, 193.4)
- moved SW2 179.4 mm to (512.7, 193.4)
- moved SW4 179.3 mm to (541.7, 193.4)
- moved U6 160.0 mm to (328.9, 313.7), turned to 90 degrees
- moved R24 151.7 mm to (349.5, 325.3), turned to -90 degrees
- moved C57 150.6 mm to (361.1, 319.5), turned to 180 degrees
- moved U9 145.8 mm to (355.4, 322.5)
- moved J3 121.2 mm to (348.9, 319.7), turned to -90 degrees
- moved R16 118.1 mm to (348.9, 303.3), turned to 90 degrees
- moved R15 113.2 mm to (353.7, 301.1)
- moved C3 111.6 mm to (326.6, 309.2), turned to 180 degrees
- moved Q1 110.1 mm to (352.0, 304.1), turned to 180 degrees
- moved U7 105.8 mm to (367.0, 305.8)
- moved C20 100.7 mm to (373.1, 304.4), turned to -90 degrees
- moved R13 96.3 mm to (368.1, 315.4), turned to 180 degrees
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Connections:
- J3 pad 2: /UART_RX -> /SWDIO
- J3 pad 3: /UART_TX -> /SWCLK
- J5 pad 1: GND -> /AIR_SENSOR_1
- J5 pad 2: /AIR_SENSOR_5 -> /AIR_SENSOR_3
- J5 pad 3: /AIR_SENSOR_3 -> /AIR_SENSOR_5
- J5 pad 4: /AIR_SENSOR_1 -> /AIR_LED_0
- J5 pad 5: /AIR_LED_0 -> /AIR_LED_2
- J5 pad 6: /AIR_LED_2 -> /AIR_LED_4
- J5 pad 7: /AIR_LED_4 -> /RIGHT_RGB_DO
- J5 pad 8: +3V3 -> unconnected-(J5-Pad8)
- J5 pad 9: +5V -> +3V3
- J6 pad 1: GND -> +5V
- J6 pad 2: /AIR_LED_5 -> +5V
- J6 pad 3: /AIR_LED_3 -> +5V
- J6 pad 4: /AIR_LED_1 -> unconnected-(J6-Pad4)
- J6 pad 5: /AIR_SENSOR_0 -> GND
- J6 pad 6: /AIR_SENSOR_2 -> GND
- J6 pad 7: /AIR_SENSOR_4 -> unconnected-(J6-Pad7)
- J6 pad 9: +5V -> +3V3
- U5 pad 12: /AIR_LED_0 -> /AIR_LED_4
- U5 pad 13: /AIR_LED_1 -> /AIR_LED_2
- U5 pad 14: /AIR_LED_2 -> /AIR_LED_0
- U5 pad 15: /AIR_LED_3 -> /AIR_LED_5
- U5 pad 16: /AIR_LED_4 -> /AIR_LED_3
- U5 pad 17: /AIR_LED_5 -> /AIR_LED_1
- U5 pad 18: /MUX_0 -> unconnected-(U5-Pad18)
- U5 pad 2: /UART_TX -> unconnected-(U5-Pad2)
- U5 pad 27: /MUX_1 -> /MUX_0
- U5 pad 28: /MUX_2 -> /MUX_1
- U5 pad 29: unconnected-(U5-Pad29) -> /MUX_2
- U5 pad 3: /UART_RX -> unconnected-(U5-Pad3)
- U9 pad 1: /AIR_SENSOR_4 -> /AIR_SENSOR_5
- U9 pad 12: /AIR_SENSOR_3 -> unconnected-(U9-Pad12)
- U9 pad 13: /AIR_SENSOR_0 -> /AIR_SENSOR_4
- U9 pad 14: /AIR_SENSOR_1 -> /AIR_SENSOR_2
- U9 pad 15: /AIR_SENSOR_2 -> /AIR_SENSOR_0
- U9 pad 2: unconnected-(U9-Pad2) -> /AIR_SENSOR_3
- U9 pad 5: /AIR_SENSOR_5 -> /AIR_SENSOR_1
Routing:
- net /SW_FUNCTION: track 0.00 -> 676.5 mm, vias 0 -> 2
- net /SW_SVC: track 0.00 -> 662.6 mm, vias 0 -> 2
- net /SW_TEST: track 0.00 -> 648.3 mm, vias 0 -> 2
- net /USB_D-: track 5.15 -> 635.7 mm, vias 0 -> 2
- net /USB_D+: track 5.13 -> 635.3 mm, vias 0 -> 2
- net +5V: track 711.2 -> 1294.5 mm, vias 1 -> 12
- net /AUX_POWER_DETECT: track 5.99 -> 558.3 mm, vias 0 -> 2
- net /RIGHT_RGB_DO: track 0.00 -> 499.8 mm, vias 0 -> 2
- net /SDA: track 8.93 -> 362.9 mm, vias 0 -> 3
- net /SCL: track 17.8 -> 366.6 mm, vias 0 -> 5
- net /AIR_LED_5: track 0.00 -> 328.8 mm, vias 0 -> 2
- net /AIR_LED_3: track 0.00 -> 326.9 mm, vias 0 -> 2
- net /AIR_LED_1: track 0.00 -> 325.0 mm, vias 0 -> 2
- net /AIR_SENSOR_4: track 0.00 -> 294.4 mm, vias 0 -> 2
- net /AIR_SENSOR_2: track 0.00 -> 294.3 mm, vias 0 -> 2
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- added copper zone on F.Cu, net GND

Commit message: First pass of the mainboard layout is done, besides art and mounting holes
Routing:
- net +3V3: track 89.2 -> 423.9 mm
- net GND: track 290.1 -> 291.9 mm, vias 49 -> 57
- net Net-(D1-Pad2): track 39.3 -> 38.1 mm
- net +5V: track 1294.5 -> 1295.0 mm, vias 12 -> 13
- added copper zone on F.Cu, net +3V3
- added copper zone on B.Cu, net GND
Other:
- board outline added: 512.3 x 155.9 mm

Commit message: Added JLCPCB part number mappings for everything, so we can export this via the jlcpcb plugin to order, once everything is finalized.
Parts:
- C1, C10, C15, C16, C2, C3, C4, C5, C6, C7, C73, C8, C9: footprint Capacitor_SMD:C_0201_0603Metric -> Capacitor_SMD:C_0402_1005Metric
- C13, C14: value 22u -> 10u; footprint Capacitor_Tantalum_SMD:CP_EIA-1608-08_AVX-J -> Capacitor_SMD:C_0805_2012Metric
- C23, C24: value 27p -> 30pF
- C57: footprint Capacitor_SMD:C_0603_1608Metric -> Capacitor_SMD:C_0402_1005Metric
- R12: value 1.7k -> 1k
- R14: value 3.3k -> 2k
- U1: value AMS1117-3.3 -> NCP1117-3.3_SOT223
- moved J5 8.09 mm to (162.3, 308.4)
- moved J6 7.26 mm to (649.3, 312.4)
- moved C5 0.46 mm to (364.8, 312.9)
- moved U1 0.30 mm to (403.6, 192.3)
- moved C14 0.25 mm to (398.8, 196.5)
- moved C9 0.23 mm to (349.8, 312.0)
- moved C13 0.22 mm to (408.7, 197.0)
- moved C16 0.22 mm to (364.4, 315.9)
- moved C3 0.14 mm to (326.5, 309.2)
- moved C11 0.09 mm to (257.4, 304.4)
- moved C12 0.08 mm to (431.8, 304.4)
Routing:
- net /RIGHT_RGB_DO: track 499.8 -> 484.4 mm
- net +5V: track 1295.0 -> 1281.0 mm, vias 13 -> 11
- net /AIR_SENSOR_5: track 201.7 -> 193.6 mm
- net /AIR_SENSOR_3: track 201.6 -> 193.5 mm
- net /AIR_SENSOR_1: track 201.1 -> 193.0 mm
- net /AIR_LED_4: track 200.9 -> 192.8 mm
- net /AIR_LED_2: track 200.3 -> 192.2 mm
- net /AIR_LED_0: track 199.7 -> 191.6 mm
- net /AIR_SENSOR_4: track 294.4 -> 287.1 mm
- net /AIR_SENSOR_2: track 294.3 -> 287.1 mm
- net /AIR_SENSOR_0: track 294.3 -> 287.0 mm
- net /AIR_LED_5: track 328.8 -> 321.5 mm
- net /AIR_LED_3: track 326.9 -> 319.6 mm
- net /AIR_LED_1: track 325.0 -> 317.7 mm
- net /SLIDER_RGB_DO: track 46.8 -> 39.6 mm
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Other:
- board size 512.3 x 155.9 mm -> 496.2 x 155.9 mm

Commit message: v0.1 of the slider PCB is likely complete, waiting for a prototype order to arrive before making any real changes.
Parts:
- added G***: LOGO, Skogaslider_Custom_Footprints:skogacons_logo, B.Cu at (575.2, 255.4)
- added H1: MountingHole, MountingHole:MountingHole_3.2mm_M3, F.Cu at (176.3, 192.5)
- added H10: MountingHole, MountingHole:MountingHole_3.2mm_M3, F.Cu at (451.9, 329.0)
- added H11: MountingHole, MountingHole:MountingHole_3.2mm_M3, F.Cu at (543.8, 329.0)
- added H12: MountingHole, MountingHole:MountingHole_3.2mm_M3, F.Cu at (635.6, 329.0)
- added H2: MountingHole, MountingHole:MountingHole_3.2mm_M3, F.Cu at (268.2, 192.5)
- added H3: MountingHole, MountingHole:MountingHole_3.2mm_M3, F.Cu at (360.0, 192.5)
- added H4: MountingHole, MountingHole:MountingHole_3.2mm_M3, F.Cu at (451.9, 192.5)
- added H5: MountingHole, MountingHole:MountingHole_3.2mm_M3, F.Cu at (543.8, 192.5)
- added H6: MountingHole, MountingHole:MountingHole_3.2mm_M3, F.Cu at (635.6, 192.5)
- added H7: MountingHole, MountingHole:MountingHole_3.2mm_M3, F.Cu at (176.3, 329.0)
- added H8: MountingHole, MountingHole:MountingHole_3.2mm_M3, F.Cu at (268.2, 329.0)
- added H9: MountingHole, MountingHole:MountingHole_3.2mm_M3, F.Cu at (360.0, 329.0)
- moved SW4 55.7 mm to (486.0, 193.4)
- moved SW3 51.5 mm to (475.7, 193.4)
- moved SW2 47.3 mm to (465.4, 193.4)
Routing:
- net /SW_FUNCTION: track 676.5 -> 622.5 mm
- net /SW_SVC: track 662.6 -> 612.0 mm
- net /SW_TEST: track 648.3 -> 601.5 mm
- net /RIGHT_RGB_DO: track 484.4 -> 493.7 mm
- net GND: track 292.2 -> 290.0 mm
Other:
- outline, holes or cut-outs redrawn
- board text added: "SKOGASLIDER - A controller for touch and air-based rhythm games skogacons 2022"

Commit message: New revision of the mainboard schematic and layout. Switched the air towers from HDMI to USB-C, and made them use the I2C bus for communication to reduce the number of pins
Parts:
- removed C57: 100nF, Capacitor_SMD:C_0402_1005Metric
- removed H11, H12, H7, H8: MountingHole, MountingHole:MountingHole_3.2mm_M3
- removed R24: 10k, Resistor_SMD:R_0603_1608Metric
- removed SW1, SW2, SW3, SW4: SW_Push, TS-1187A-B-A-B:SW_TS-1187A-B-A-B
- removed TP1, TP2, TP3, TP4: TestPoint, TestPoint:TestPoint_Pad_D1.5mm
- removed U9: 74HC4051, Package_SO:TSSOP-16_4.4x5mm_P0.65mm
- added S1: TS-1187A-B-A-B, TS-1187A-B-A-B:TS1187ABAB, F.Cu at (335.8, 348.2)
- H1, H10, H2, H3, H4, H5, H6, H9: value MountingHole -> MountingHole_Pad; footprint MountingHole:MountingHole_3.2mm_M3 -> MountingHole:MountingHole_3.2mm_M3_DIN965_Pad_TopBottom
- J5, J6: value HDMI_A_No_Video -> USB_C_Receptacle_USB2.0; footprint Skogaslider_Custom_Footprints:HDMI_Connector_SMD -> Connector_USB:USB_C_Receptacle_HRO_TYPE-C-31-M-12
- moved H5 320.3 mm to (271.3, 361.1)
- moved H2 282.0 mm to (547.3, 232.8)
- moved C13 216.5 mm to (252.6, 346.9)
- moved H9 212.7 mm to (170.3, 232.8)
- moved U1 210.4 mm to (259.3, 345.5), turned to 0 degrees
- moved H10 204.6 mm to (271.3, 232.8)
- moved C14 200.1 mm to (266.3, 346.5)
- moved H6 190.3 mm to (547.3, 361.1)
- moved H1 168.6 mm to (170.3, 361.1)
- moved H4 168.6 mm to (446.3, 361.1)
- moved J6 108.5 mm to (576.3, 232.2), turned to 180 degrees
- moved H3 95.2 mm to (446.3, 232.8)
- moved J5 79.1 mm to (141.3, 232.2), turned to 180 degrees
- moved R12 74.6 mm to (365.0, 238.6), turned to 0 degrees
- moved R6 71.2 mm to (341.7, 240.3)
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Connections:
- R12 pad 1: Net-(D2-Pad2) -> +5V
- U5 pad 11: /SW_FUNCTION -> unconnected-(U5-Pad11)
- U5 pad 12: /AIR_LED_4 -> unconnected-(U5-Pad12)
- U5 pad 13: /AIR_LED_2 -> unconnected-(U5-Pad13)
- U5 pad 14: /AIR_LED_0 -> unconnected-(U5-Pad14)
- U5 pad 15: /AIR_LED_5 -> unconnected-(U5-Pad15)
- U5 pad 16: /AIR_LED_3 -> unconnected-(U5-Pad16)
- U5 pad 17: /AIR_LED_1 -> unconnected-(U5-Pad17)
- U5 pad 27: /MUX_0 -> unconnected-(U5-Pad27)
- U5 pad 28: /MUX_1 -> unconnected-(U5-Pad28)
- U5 pad 29: /MUX_2 -> unconnected-(U5-Pad29)
- U5 pad 38: /AIR_SENSOR_IN -> unconnected-(U5-Pad38)
- U5 pad 8: /SW_TEST -> unconnected-(U5-Pad8)
- U5 pad 9: /SW_SVC -> unconnected-(U5-Pad9)
Routing:
- net /SW_FUNCTION: track 622.5 -> 0.00 mm, vias 2 -> 0
- net /SW_SVC: track 612.0 -> 0.00 mm, vias 2 -> 0
- net /SW_TEST: track 601.5 -> 0.00 mm, vias 2 -> 0
- net /SCL: track 366.6 -> 772.4 mm, vias 5 -> 9
- net /SDA: track 362.9 -> 761.9 mm, vias 3 -> 11
- net +3V3: track 419.0 -> 84.1 mm, vias 0 -> 2
- net /AIR_LED_5: track 321.5 -> 0.00 mm, vias 2 -> 0
- net /AIR_LED_3: track 319.6 -> 0.00 mm, vias 2 -> 0
- net /AIR_LED_1: track 317.7 -> 0.00 mm, vias 2 -> 0
- net /AIR_SENSOR_4: track 287.1 -> 0.00 mm, vias 2 -> 0
- net /AIR_SENSOR_2: track 287.1 -> 0.00 mm, vias 2 -> 0
- net /AIR_SENSOR_0: track 287.0 -> 0.00 mm, vias 2 -> 0
- net /AIR_SENSOR_5: track 193.6 -> 0.00 mm, vias 2 -> 0
- net /AIR_SENSOR_3: track 193.5 -> 0.00 mm, vias 2 -> 0
- net /AIR_SENSOR_1: track 193.0 -> 0.00 mm, vias 2 -> 0
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Other:
- board size 496.2 x 155.9 mm -> 475 x 140.3 mm
- board text added: "SKOGASLIDER - A controller for touch and air-based rhythm games skogacons 2023"
- board text removed: "SKOGASLIDER - A controller for touch and air-based rhythm games skogacons 2022"

Commit message: Fix up the top edge of the board so it fits within the controller CAD, and add more mounting holes.
Parts:
- removed J3: Conn_01x03, Connector_PinHeader_2.54mm:PinHeader_1x03_P2.54mm_Vertical
- added H7: MountingHole_Pad, MountingHole:MountingHole_3.2mm_M3_DIN965_Pad_TopBottom, F.Cu at (358.8, 361.1)
- added H8: MountingHole_Pad, MountingHole:MountingHole_3.2mm_M3_DIN965_Pad_TopBottom, F.Cu at (358.8, 232.8)
- added TP1: TestPoint, TestPoint:TestPoint_Pad_1.0x1.0mm, F.Cu at (296.7, 361.9)
- added TP2: TestPoint, TestPoint:TestPoint_Pad_1.0x1.0mm, F.Cu at (299.3, 361.9)
- added TP3: TestPoint, TestPoint:TestPoint_Pad_1.0x1.0mm, F.Cu at (301.8, 361.9)
Routing:
- net +5V: track 1470.9 -> 1472.5 mm
Other:
- board size 475 x 140.3 mm -> 475 x 139.9 mm
