File: KiCAD Projects/skogaslider-main-pcb/skogaslider-main-pcb.kicad_pcb (KiCad board)
At the start: 2 copper layers, 475 x 139.9 mm, 174 parts, among them J1 USB_C_Receptacle_USB2.0, J2 USB_C_Receptacle_USB2.0, J4 Conn_02x16_Top_Bottom, J5 USB_C_Receptacle_USB2.0, J6 USB_C_Receptacle_USB2.0, Q1 BSS138, U1 NCP1117-3.3_SOT223, U2 MPR121QR2, U3 MPR121QR2, U4 USBLC6-2P6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

Commit message: Minor revision of the slider PCB to re-arrange the mounting holes to fit the CAD better.
Parts:
- added H11: MountingHole_Pad, MountingHole:MountingHole_3.2mm_M3_DIN965_Pad_TopBottom, F.Cu at (416.8, 232.8)
- moved H8 58.0 mm to (300.8, 232.8)
Changed lines of the file:
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@@
   (net 172 "unconnected-(H7-Pad1)")
   (net 173 "unconnected-(H8-Pad1)")
+  (net 174 "unconnected-(H11-Pad1)")
   (footprint "WS2812B-4020:WS2812B-4020" (layer "F.Cu")
     (at 445.821075 333.191669)
@@
     )
   )
+  (footprint "MountingHole:MountingHole_3.2mm_M3_DIN965_Pad_TopBottom" (layer "F.Cu")
+    (at 416.8 232.78)
+    (descr "Mounting Hole 3.2mm, M3, DIN965")
+    (tags "mounting hole 3.2mm m3 din965")
+    (property "Sheetfile" "skogaslider-main-pcb.kicad_sch")
+    (property "Sheetname" "")
+    (attr exclude_from_pos_files)
+    (fp_text reference "H11" (at 0 -3.8) (layer "F.SilkS")
+      (effects (font (size 1 1) (thickness 0.15)))
+    )
+    (fp_text value "MountingHole_Pad" (at 0 3.8) (layer "F.Fab")
+      (effects (font (size 1 1) (thickness 0.15)))
+    )
+    (fp_text user "${REFERENCE}" (at 0 0) (layer "F.Fab")
+      (effects (font (size 1 1) (thickness 0.15)))
+    )
+    (fp_circle (center 0 0) (end 2.8 0) (layer "Cmts.User") (width 0.15) (fill none))
+    (fp_circle (center 0 0) (end 3.05 0) (layer "F.CrtYd") (width 0.05) (fill none))
+    (pad "1" thru_hole circle (at 0 0) (size 3.6 3.6) (drill 3.2) (layers *.Cu *.Mask)
+      (net 174 "unconnected-(H11-Pad1)") (pinfunction "1") (pintype "input+no_connect"))
+    (pad "1" connect circle (at 0 0) (size 5.6 5.6) (layers "F.Cu" "F.Mask")
+      (net 174 "unconnected-(H11-Pad1)") (pinfunction "1") (pintype "input+no_connect"))
+    (pad "1" connect circle (at 0 0) (size 5.6 5.6) (layers "B.Cu" "B.Mask")
+      (net 174 "unconnected-(H11-Pad1)") (pinfunction "1") (pintype "input+no_connect"))
+  )
   (footprint "RP2040_minimal:RP2040-QFN-56" (layer "F.Cu")
     (at 310.592346 353.631669 -90)
@@
     )
   )
+  (footprint "MountingHole:MountingHole_3.2mm_M3_DIN965_Pad_TopBottom" (layer "F.Cu")
+    (at 300.8 232.78)
+    (descr "Mounting Hole 3.2mm, M3, DIN965")
+    (tags "mounting hole 3.2mm m3 din965")
+    (property "Sheetfile" "skogaslider-main-pcb.kicad_sch")
+    (property "Sheetname" "")
+    (attr exclude_from_pos_files)
+    (fp_text reference "H8" (at 0 -3.8) (layer "F.SilkS")
+      (effects (font (size 1 1) (thickness 0.15)))
+    )
+    (fp_text value "MountingHole_Pad" (at 0 3.8) (layer "F.Fab")
+      (effects (font (size 1 1) (thickness 0.15)))
+    )
+    (fp_text user "${REFERENCE}" (at 0 0) (layer "F.Fab")
+      (effects (font (size 1 1) (thickness 0.15)))
+    )
+    (fp_circle (center 0 0) (end 2.8 0) (layer "Cmts.User") (width 0.15) (fill none))
+    (fp_circle (center 0 0) (end 3.05 0) (layer "F.CrtYd") (width 0.05) (fill none))
+    (pad "1" connect circle (at 0 0) (size 5.6 5.6) (layers "F.Cu" "F.Mask")
+      (net 173 "unconnected-(H8-Pad1)") (pinfunction "1") (pintype "input+no_connect"))
+    (pad "1" thru_hole circle (at 0 0) (size 3.6 3.6) (drill 3.2) (layers *.Cu *.Mask)
+      (net 173 "unconnected-(H8-Pad1)") (pinfunction "1") (pintype "input+no_connect"))
+    (pad "1" connect circle (at 0 0) (size 5.6 5.6) (layers "B.Cu" "B.Mask")
+      (net 173 "unconnected-(H8-Pad1)") (pinfunction "1") (pintype "input+no_connect"))
+  )
   (footprint "WS2812B-4020:WS2812B-4020" (layer "F.Cu")
     (at 426.487743 333.191669)
@@
       (net 92 "Net-(D42-Pad2)") (pinfunction "DIN") (pintype "input"))
   )
-  (footprint "MountingHole:MountingHole_3.2mm_M3_DIN965_Pad_TopBottom" (layer "F.Cu")
-    (at 358.81 232.78)
-    (descr "Mounting Hole 3.2mm, M3, DIN965")
-    (tags "mounting hole 3.2mm m3 din965")
-    (property "Sheetfile" "skogaslider-main-pcb.kicad_sch")
-    (property "Sheetname" "")
-    (attr exclude_from_pos_files)
-    (fp_text reference "H8" (at 0 -3.8) (layer "F.SilkS") hide
-      (effects (font (size 1 1) (thickness 0.15)))
-    )
-    (fp_text value "MountingHole_Pad" (at 0 3.8) (layer "F.Fab")
-      (effects (font (size 1 1) (thickness 0.15)))
-    )
-    (fp_text user "${REFERENCE}" (at 0 0) (layer "F.Fab")
-      (effects (font (size 1 1) (thickness 0.15)))
-    )
-    (fp_circle (center 0 0) (end 2.8 0) (layer "Cmts.User") (width 0.15) (fill none))
-    (fp_circle (center 0 0) (end 3.05 0) (layer "F.CrtYd") (width 0.05) (fill none))
-    (pad "1" connect circle (at 0 0) (size 5.6 5.6) (layers "F.Cu" "F.Mask")
-      (net 173 "unconnected-(H8-Pad1)") (pinfunction "1") (pintype "input+no_connect"))
-    (pad "1" thru_hole circle (at 0 0) (size 3.6 3.6) (drill 3.2) (layers *.Cu *.Mask)
-      (net 173 "unconnected-(H8-Pad1)") (pinfunction "1") (pintype "input+no_connect"))
-    (pad "1" connect circle (at 0 0) (size 5.6 5.6) (layers "B.Cu" "B.Mask")
-      (net 173 "unconnected-(H8-Pad1)") (pinfunction "1") (pintype "input+no_connect"))
-  )
   (footprint "Capacitor_SMD:C_0402_1005Metric" (layer "F.Cu")
