File: KiCAD Projects/skogaslider-main-pcb/skogaslider-main-pcb.kicad_sch (KiCad schematic)
At the start: 170 parts, among them J2 USB_C_Receptacle_USB2.0, J3 Conn_02x16_Top_Bottom, U1 W25Q128JVS, U2 USBLC6-2P6, U3 RP2040, U4 MPR121QR2, U5 AMS1117-3.3, U6 MPR121QR2, U7 MPR121QR2, Y1 ABLS-12.000MHZ-B4-T

Commit message: Almost final schematic for the main slider, minus a couple of small tweaks. Significant progress on slider board layout. MPR121 layouts are essentially complete minus the key wiring. USB C ports and LEDs are also laid out.
Parts:
- removed C26, C27, C28, C30, C32, C33, C34, C36, C38, C39, C40, C57: 100nF, symbol Device:C
- removed D10, D12, D14, D15, D16, D18, D2, D3, D4, D6, D8, D9: WS2812B, LED_SMD:LED_WS2812B_PLCC4_5.0x5.0mm_P3.2mm, symbol LED:WS2812B
- removed SW? (x4): SW_Push, symbol Switch:SW_Push
- added C41, C43, C47, C49, C53, C55, C59, C61, C65, C67, C71, C72: 100nF, Capacitor_SMD:C_0402_1005Metric, symbol Device:C
- added C57: 100nF, Capacitor_SMD:C_0603_1608Metric, symbol Device:C_Small
- added D19, D23, D25, D29, D31, D35, D37, D41, D43, D47, D48, D49: WS2812B, WS2812B-4020:WS2812B-4020, symbol LED:WS2812B
- added R12: 1.7k, Resistor_SMD:R_0603_1608Metric, symbol Device:R
- added R14: 3.3k, Resistor_SMD:R_0603_1608Metric, symbol Device:R
- added R21: 50k, Resistor_SMD:R_0603_1608Metric, symbol Device:R
- added R24: 10k, Resistor_SMD:R_0603_1608Metric, symbol Device:R
- added U9: 74HC4051, Package_SO:TSSOP-16_4.4x5mm_P0.65mm, symbol 74xx:74HC4051
- C11: renamed from C21; footprint (none) -> Capacitor_SMD:C_0402_1005Metric
- C12: renamed from C24; footprint (none) -> Capacitor_SMD:C_0402_1005Metric
- C17: renamed from C5; footprint (none) -> Capacitor_SMD:C_0402_1005Metric
- C18: renamed from C19; footprint (none) -> Capacitor_SMD:C_0402_1005Metric
- C19: renamed from C23; footprint (none) -> Capacitor_SMD:C_0402_1005Metric
- C21: renamed from C22; footprint (none) -> Capacitor_SMD:C_0402_1005Metric
- C22: renamed from C20; footprint (none) -> Capacitor_SMD:C_0402_1005Metric
- C25, C42, C44, C45, C46, C48, C50, C51, C52, C54, C56, C58, C60, C62, C63, C64, C66, C68, C69, C70: footprint (none) -> Capacitor_SMD:C_0402_1005Metric
- C26: renamed from C29; footprint (none) -> Capacitor_SMD:C_0402_1005Metric
- C27: renamed from C31; footprint (none) -> Capacitor_SMD:C_0402_1005Metric
- C28: renamed from C35; footprint (none) -> Capacitor_SMD:C_0402_1005Metric
- C29: renamed from C37; footprint (none) -> Capacitor_SMD:C_0402_1005Metric
- C30: renamed from C41; footprint (none) -> Capacitor_SMD:C_0402_1005Metric
- C31: renamed from C43; footprint (none) -> Capacitor_SMD:C_0402_1005Metric
- C32: renamed from C47; footprint (none) -> Capacitor_SMD:C_0402_1005Metric
- C33: renamed from C49; footprint (none) -> Capacitor_SMD:C_0402_1005Metric
- C34: renamed from C53; footprint (none) -> Capacitor_SMD:C_0402_1005Metric
- C35: renamed from C55; footprint (none) -> Capacitor_SMD:C_0402_1005Metric
- C36: renamed from C59; footprint (none) -> Capacitor_SMD:C_0402_1005Metric
- C37: renamed from C61; footprint (none) -> Capacitor_SMD:C_0402_1005Metric
- C38: renamed from C65; footprint (none) -> Capacitor_SMD:C_0402_1005Metric
- C39: renamed from C67; footprint (none) -> Capacitor_SMD:C_0402_1005Metric
- C40: renamed from C71; footprint (none) -> Capacitor_SMD:C_0402_1005Metric
- D10: renamed from D23; footprint LED_SMD:LED_WS2812B_PLCC4_5.0x5.0mm_P3.2mm -> WS2812B-4020:WS2812B-4020
- D11: renamed from D25; footprint LED_SMD:LED_WS2812B_PLCC4_5.0x5.0mm_P3.2mm -> WS2812B-4020:WS2812B-4020
- D12: renamed from D29; footprint LED_SMD:LED_WS2812B_PLCC4_5.0x5.0mm_P3.2mm -> WS2812B-4020:WS2812B-4020
- D13: renamed from D31; footprint LED_SMD:LED_WS2812B_PLCC4_5.0x5.0mm_P3.2mm -> WS2812B-4020:WS2812B-4020
- D14: renamed from D35; footprint LED_SMD:LED_WS2812B_PLCC4_5.0x5.0mm_P3.2mm -> WS2812B-4020:WS2812B-4020
- D15: renamed from D37; footprint LED_SMD:LED_WS2812B_PLCC4_5.0x5.0mm_P3.2mm -> WS2812B-4020:WS2812B-4020
- D16: renamed from D41; footprint LED_SMD:LED_WS2812B_PLCC4_5.0x5.0mm_P3.2mm -> WS2812B-4020:WS2812B-4020
- D17: renamed from D43; footprint LED_SMD:LED_WS2812B_PLCC4_5.0x5.0mm_P3.2mm -> WS2812B-4020:WS2812B-4020
- D18: renamed from D47; footprint LED_SMD:LED_WS2812B_PLCC4_5.0x5.0mm_P3.2mm -> WS2812B-4020:WS2812B-4020
- D20, D21, D22, D24, D26, D27, D28, D30, D32, D33, D34, D36, D38, D39, D40, D42, D44, D45, D46: footprint LED_SMD:LED_WS2812B_PLCC4_5.0x5.0mm_P3.2mm -> WS2812B-4020:WS2812B-4020
- D3: renamed from D1; footprint LED_SMD:LED_WS2812B_PLCC4_5.0x5.0mm_P3.2mm -> WS2812B-4020:WS2812B-4020
- D4: renamed from D5; footprint LED_SMD:LED_WS2812B_PLCC4_5.0x5.0mm_P3.2mm -> WS2812B-4020:WS2812B-4020
- D5: renamed from D7; footprint LED_SMD:LED_WS2812B_PLCC4_5.0x5.0mm_P3.2mm -> WS2812B-4020:WS2812B-4020
- D6: renamed from D11; footprint LED_SMD:LED_WS2812B_PLCC4_5.0x5.0mm_P3.2mm -> WS2812B-4020:WS2812B-4020
- D7: renamed from D13; footprint LED_SMD:LED_WS2812B_PLCC4_5.0x5.0mm_P3.2mm -> WS2812B-4020:WS2812B-4020
- D8: renamed from D17; footprint LED_SMD:LED_WS2812B_PLCC4_5.0x5.0mm_P3.2mm -> WS2812B-4020:WS2812B-4020
- D9: renamed from D19; footprint LED_SMD:LED_WS2812B_PLCC4_5.0x5.0mm_P3.2mm -> WS2812B-4020:WS2812B-4020
- J1: renamed from J?; footprint (none) -> Connector_USB:USB_C_Receptacle_HRO_TYPE-C-31-M-12
- J2: footprint (none) -> Connector_USB:USB_C_Receptacle_HRO_TYPE-C-31-M-12
- J3: renamed from J?; footprint (none) -> Connector_PinHeader_2.54mm:PinHeader_1x05_P2.54mm_Vertical
- J7, J8: renamed from J?; footprint (none) -> Connector_JST:JST_PH_S4B-PH-K_1x04_P2.00mm_Horizontal
- R1: renamed from R10; footprint (none) -> Resistor_SMD:R_0603_1608Metric
- R10: renamed from R14; footprint (none) -> Resistor_SMD:R_0603_1608Metric
- R11: renamed from R4; footprint Capacitor_SMD:C_0402_1005Metric -> Resistor_SMD:R_0603_1608Metric
- R13: renamed from R5; footprint Capacitor_SMD:C_0402_1005Metric -> Resistor_SMD:R_0603_1608Metric
- R15, R16, R7, R8: renamed from R?; footprint (none) -> Resistor_SMD:R_0603_1608Metric
- R17: renamed from R2; value DNF -> 10k; footprint Capacitor_SMD:C_0402_1005Metric -> Resistor_SMD:R_0603_1608Metric
- R18: renamed from R11; footprint (none) -> Resistor_SMD:R_0603_1608Metric
- R19: renamed from R13; footprint (none) -> Resistor_SMD:R_0603_1608Metric
- R2: renamed from R12; footprint (none) -> Resistor_SMD:R_0603_1608Metric
- R20: renamed from R1; footprint Capacitor_SMD:C_0402_1005Metric -> Resistor_SMD:R_0402_1005Metric
- R22: renamed from R9; footprint (none) -> Resistor_SMD:R_0603_1608Metric
- R23: renamed from R3; footprint Capacitor_SMD:C_0402_1005Metric -> Resistor_SMD:R_0402_1005Metric
- R3: renamed from R15; footprint (none) -> Resistor_SMD:R_0603_1608Metric
- R4: renamed from R16; footprint (none) -> Resistor_SMD:R_0603_1608Metric
- R5: renamed from R6; footprint (none) -> Resistor_SMD:R_0603_1608Metric
- R6: renamed from R7; footprint (none) -> Resistor_SMD:R_0603_1608Metric
- R9: renamed from R8; footprint (none) -> Resistor_SMD:R_0603_1608Metric
- SW1, SW2, SW3, SW4: renamed from SW?; footprint (none) -> TS-1187A-B-A-B:SW_TS-1187A-B-A-B
- TP1, TP2, TP3, TP4: footprint (none) -> TestPoint:TestPoint_Pad_D1.5mm
- gave numbers to parts that had none: 6
- renumbered C6 to C1, C17 to C10, C3 to C13, C18 to C14, C8 to C15, C10 to C16, C7 to C2, C4 to C20, C1 to C23, C2 to C24, C14 to C3, C9 to C4, C11 to C5, C12 to C6, C13 to C7, C15 to C8, C16 to C9, J3 to J4, U5 to U1, U4 to U2, U7 to U3, U2 to U4, U3 to U5, U1 to U7, U6 to U8
Connections:
- net SW_BRIGHTNESS_UP is gone; now on net SW_SVC: U5.9 (GPIO7)
- net SW_COIN is gone; now on net AIR_LED_2: U5.14 (GPIO11)
- net +3V3: now also C57.2, R21.1, U9.16 (VCC); no longer U3.4 (ADDR)
- net +5V: now also C17.2, U4.5 (VBUS), C41.1, C43.1, C47.1, C49.1, C53.1, C55.1, C59.1, C61.1, C65.1, C67.1, C71.1, C72.1, D19.1 (VDD), D23.1 (VDD), D25.1 (VDD), D29.1 (VDD), D31.1 (VDD), D35.1 (VDD), D37.1 (VDD), D41.1 (VDD), D43.1 (VDD), D47.1 (VDD), D48.1 (VDD), D49.1 (VDD), R12.1
- net AIR_LED_0: now also U5.12 (GPIO9); no longer U5.15 (GPIO12)
- net AIR_LED_1: now also U5.13 (GPIO10); no longer U5.16 (GPIO13)
- net AIR_LED_2: no longer U5.17 (GPIO14)
- net AIR_LED_3: now also U5.15 (GPIO12); no longer U5.18 (GPIO15)
- net AIR_LED_4: now also U5.16 (GPIO13); no longer U5.27 (GPIO16)
- net AIR_LED_5: now also U5.17 (GPIO14); no longer U5.28 (GPIO17)
- net AIR_SENSOR_0: now also U9.13 (A0); no longer U5.29 (GPIO18)
- net AIR_SENSOR_1: now also U9.14 (A1); no longer U5.30 (GPIO19)
- net AIR_SENSOR_2: now also U9.15 (A2); no longer U5.31 (GPIO20)
- net AIR_SENSOR_3: now also U9.12 (A3); no longer U5.32 (GPIO21)
- net AIR_SENSOR_4: now also U9.1 (A4); no longer U5.34 (GPIO22)
- net AIR_SENSOR_5: now also U9.5 (A5); no longer U5.35 (GPIO23)
- net GND: now also C41.2, C43.2, C47.2, C49.2, C53.2, C55.2, C57.1, C59.2, C61.2, C65.2, C67.2, C71.2, C72.2, D19.3 (VSS), D23.3 (VSS), D25.3 (VSS), D29.3 (VSS), D31.3 (VSS), D35.3 (VSS), D37.3 (VSS), D41.3 (VSS), D43.3 (VSS), D47.3 (VSS), D48.3 (VSS), D49.3 (VSS), R14.2, R24.2, U9.7 (VEE), U9.8 (GND)
- net KEY_1: now also U2.19 (LED7/ELE11); no longer U2.8 (ELE0)
- net KEY_10: now also U2.10 (ELE2); no longer U2.17 (LED5/ELE9)
- net KEY_11: now also U2.9 (ELE1); no longer U2.18 (LED6/ELE10)
- net KEY_12: now also U2.8 (ELE0); no longer U2.19 (LED7/ELE11)
- net KEY_13: now also U3.19 (LED7/ELE11); no longer U3.8 (ELE0)
- net KEY_14: now also U3.18 (LED6/ELE10); no longer U3.9 (ELE1)
- net KEY_15: now also U3.17 (LED5/ELE9); no longer U3.10 (ELE2)
- net KEY_16: now also U3.16 (LED4/ELE8); no longer U3.11 (ELE3)
- net KEY_17: now also U3.15 (LED3/ELE7); no longer U3.12 (LED0/ELE4)
- net KEY_18: now also U3.14 (LED2/ELE6); no longer U3.13 (LED1/ELE5)
- net KEY_19: now also U3.13 (LED1/ELE5); no longer U3.14 (LED2/ELE6)
- net KEY_2: now also U2.18 (LED6/ELE10); no longer U2.9 (ELE1)
- net KEY_20: now also U3.12 (LED0/ELE4); no longer U3.15 (LED3/ELE7)
- net KEY_21: now also U3.11 (ELE3); no longer U3.16 (LED4/ELE8)
- net KEY_22: now also U3.10 (ELE2); no longer U3.17 (LED5/ELE9)
- net KEY_23: now also U3.9 (ELE1); no longer U3.18 (LED6/ELE10)
- net KEY_24: now also U3.8 (ELE0); no longer U3.19 (LED7/ELE11)
- net KEY_25: now also U8.19 (LED7/ELE11); no longer U8.8 (ELE0)
- net KEY_26: now also U8.18 (LED6/ELE10); no longer U8.9 (ELE1)
- net KEY_27: now also U8.17 (LED5/ELE9); no longer U8.10 (ELE2)
- net KEY_28: now also U8.16 (LED4/ELE8); no longer U8.11 (ELE3)
- net KEY_29: now also U8.15 (LED3/ELE7); no longer U8.12 (LED0/ELE4)
- net KEY_3: now also U2.17 (LED5/ELE9); no longer U2.10 (ELE2)
- net KEY_30: now also U8.14 (LED2/ELE6); no longer U8.13 (LED1/ELE5)
- net KEY_31: now also U8.13 (LED1/ELE5); no longer U8.14 (LED2/ELE6)
- net KEY_32: now also U8.12 (LED0/ELE4); no longer U8.15 (LED3/ELE7)
- net KEY_4: now also U2.16 (LED4/ELE8); no longer U2.11 (ELE3)
- net KEY_5: now also U2.15 (LED3/ELE7); no longer U2.12 (LED0/ELE4)
- net KEY_6: now also U2.14 (LED2/ELE6); no longer U2.13 (LED1/ELE5)
- net KEY_7: now also U2.13 (LED1/ELE5); no longer U2.14 (LED2/ELE6)
- net KEY_8: now also U2.12 (LED0/ELE4); no longer U2.15 (LED3/ELE7)
- net KEY_9: now also U2.11 (ELE3); no longer U2.16 (LED4/ELE8)
- net RGB_LED: now also U5.4 (GPIO2); no longer U5.8 (GPIO6)
- net SCL: now also U8.4 (ADDR)
- net SDA: now also U3.4 (ADDR); no longer U8.4 (ADDR)
- net SLIDER_RGB_DO: now also D49.2 (DOUT); no longer D45.2 (DOUT)
- net SW_SVC: no longer U5.13 (GPIO10)
- net SW_TEST: now also U5.8 (GPIO6); no longer U5.12 (GPIO9)
- net USB_D+: now also U4.6 (I/O1)
- net USB_D-: now also U4.4 (I/O2)
- net at D22.2 (DOUT): now also D23.4 (DIN)
- net at D22.4 (DIN): now also D21.2 (DOUT); no longer D21.4 (DIN)
- net at D18.2 (DOUT): now also D19.4 (DIN)
- net at D46.2 (DOUT): now also D47.4 (DIN)
- net at D34.2 (DOUT): now also D35.4 (DIN)
- net at D26.2 (DOUT): now also D27.4 (DIN)
- net at D10.2 (DOUT), D11.4 (DIN): no longer D26.4 (DIN)
- net at D27.2 (DOUT): now also D28.4 (DIN); no longer D30.4 (DIN)
- net at D24.4 (DIN): now also D23.2 (DOUT); no longer D21.2 (DOUT)
- net AIR_SENSOR_IN: now reaches U5.38 (GPIO26_ADC0)
- net AIR_SENSOR_IN: now also U9.3 (A)
- net at D16.2 (DOUT), D17.4 (DIN): no longer D44.4 (DIN)
- net PRE_USB_D+: now reaches J2.A7 (D-), J2.B7 (D-), TP2.1, U4.3 (I/O2)
- net at D1.2 (A), J2.A4 (VBUS), J2.A9 (VBUS)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: no longer C17.2, U4.5 (VBUS)
- net at D8.2 (DOUT), D9.4 (DIN): no longer D20.4 (DIN)
- net at D6.4 (DIN): now also D5.2 (DOUT)
- net at D20.2 (DOUT): now also D21.4 (DIN)
- net at D14.2 (DOUT), D15.4 (DIN): no longer D38.4 (DIN)
- net at D33.2 (DOUT): now also D34.4 (DIN); no longer D36.4 (DIN)
- net PRE_USB_D-: now reaches J2.A6 (D+), J2.B6 (D+), TP3.1, U4.1 (I/O1)
- net at D12.2 (DOUT), D13.4 (DIN): no longer D32.4 (DIN)
- net at D40.2 (DOUT): now also D41.4 (DIN)
- net at D28.2 (DOUT): now also D29.4 (DIN)
- net at D38.2 (DOUT): now also D39.4 (DIN)
- net at D42.4 (DIN): now also D41.2 (DOUT); no longer D39.2 (DOUT)
- net at D32.2 (DOUT): now also D33.4 (DIN)
- net at D44.2 (DOUT): now also D45.4 (DIN)
- net RUN: no longer names the net of U5.26 (RUN)
- net RUN: now also R21.2
- net SW_BRIGHTNESS_DOWN renamed SW_FUNCTION
- net SW_FUNCTION: now also SW4.2
- net SW_TOUCH_SENS_DOWN renamed AUX_POWER_DETECT
- net AUX_POWER_DETECT: now also R12.2, R14.1
- removed net SW_TOUCH_SENS_UP: SW4.2, U5.4 (GPIO2)
- new net: D25.2 (DOUT), D26.4 (DIN)
- new net: D24.2 (DOUT), D25.4 (DIN)
- new net: D31.2 (DOUT), D32.4 (DIN)
- new net: D30.2 (DOUT), D31.4 (DIN)
- new net: D45.2 (DOUT), D46.4 (DIN)
- new net: D42.2 (DOUT), D43.4 (DIN)
- new net: D39.2 (DOUT), D40.4 (DIN)
- new net: D29.2 (DOUT), D30.4 (DIN)
- new net: D47.2 (DOUT), D48.4 (DIN)
- new net: D37.2 (DOUT), D38.4 (DIN)
- new net: D36.2 (DOUT), D37.4 (DIN)
- new net: D19.2 (DOUT), D20.4 (DIN)
- new net: D43.2 (DOUT), D44.4 (DIN)
- new net: D35.2 (DOUT), D36.4 (DIN)
- new net: D48.2 (DOUT), D49.4 (DIN)
- new net: R24.1, U9.6 (~{E})
- new net MUX_0: U5.18 (GPIO15), U9.11 (S0)
- new net MUX_1: U5.27 (GPIO16), U9.10 (S1)
- new net MUX_2: U5.28 (GPIO17), U9.9 (S2)
- no-connect marks 40 -> 29
Other:
- note added: "Air Sensor Multiplexer"
- note added: "MPR121 #2 - Address 0x5C (Keys 13-24)"
- note added: "MPR121 #3 - Address 0x5D (Keys 25-32)"
- note removed: "MPR121 #2 - Address 0x5B (Keys 13-24)"
- note removed: "MPR121 #3 - Address 0x5C (Keys 25-32)"
- moved on the sheet: C11, C12, C18, C19, C20, C21, C22, C23, C24, D2, J3, J4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

Commit message: More layout progress for the main slider PCB
Parts:
- C13, C14: footprint Capacitor_SMD:C_0805_2012Metric -> Capacitor_Tantalum_SMD:CP_EIA-1608-08_AVX-J
Connections:
- net +5V: no longer R12.1
- net at D2.2 (A), J1.A4 (VBUS), J1.A9 (VBUS)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: now also R12.1
Other:
- moved on the sheet: D2, R12, R14
Changed lines of the file:
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@@
   (junction (at 241.3 205.74) (diameter 0) (color 0 0 0 0)
   )
+  (junction (at 130.175 71.755) (diameter 0) (color 0 0 0 0)
+  )
   (junction (at 67.945 38.735) (diameter 0) (color 0 0 0 0)
   )
@@
   (junction (at 342.9 245.745) (diameter 0) (color 0 0 0 0)
   )
-  (junction (at 113.03 81.28) (diameter 0) (color 0 0 0 0)
+  (junction (at 130.175 83.82) (diameter 0) (color 0 0 0 0)
   )
   (junction (at 363.22 205.74) (diameter 0) (color 0 0 0 0)
@@
   (junction (at 261.62 220.98) (diameter 0) (color 0 0 0 0)
   )
-  (junction (at 113.03 71.755) (diameter 0) (color 0 0 0 0)
-  )
   (junction (at 322.58 245.745) (diameter 0) (color 0 0 0 0)
   )
@@
     (stroke (width 0) (type default) (color 0 0 0 0))
   )
-  (wire (pts (xy 113.03 81.28) (xy 133.35 81.28))
+  (wire (pts (xy 130.175 71.755) (xy 134.62 71.755))
+    (stroke (width 0) (type default) (color 0 0 0 0))
+  )
+  (wire (pts (xy 130.175 83.82) (xy 150.495 83.82))
     (stroke (width 0) (type default) (color 0 0 0 0))
   )
@@
     (stroke (width 0) (type default) (color 0 0 0 0))
   )
-  (wire (pts (xy 130.81 71.755) (xy 134.62 71.755))
-    (stroke (width 0) (type default) (color 0 0 0 0))
-  )
   (wire (pts (xy 329.565 88.9) (xy 329.565 90.805))
     (stroke (width 0) (type default) (color 0 0 0 0))
@@
     (stroke (width 0) (type default) (color 0 0 0 0))
   )
+  (wire (pts (xy 130.175 71.755) (xy 130.175 74.295))
+    (stroke (width 0) (type default) (color 0 0 0 0))
+  )
   (wire (pts (xy 342.9 205.74) (xy 353.06 205.74))
     (stroke (width 0) (type default) (color 0 0 0 0))
@@
     (stroke (width 0) (type default) (color 0 0 0 0))
   )
-  (wire (pts (xy 113.03 71.755) (xy 123.19 71.755))
-    (stroke (width 0) (type default) (color 0 0 0 0))
-  )
   (wire (pts (xy 373.38 205.74) (xy 373.38 209.55))
     (stroke (width 0) (type default) (color 0 0 0 0))
@@
     (stroke (width 0) (type default) (color 0 0 0 0))
   )
-  (wire (pts (xy 113.03 79.375) (xy 113.03 81.28))
+  (wire (pts (xy 130.175 81.915) (xy 130.175 83.82))
     (stroke (width 0) (type default) (color 0 0 0 0))
   )
@@
     (stroke (width 0) (type default) (color 0 0 0 0))
   )
-  (wire (pts (xy 102.235 81.28) (xy 104.14 81.28))
+  (wire (pts (xy 119.38 83.82) (xy 121.285 83.82))
     (stroke (width 0) (type default) (color 0 0 0 0))
   )
@@
     (stroke (width 0) (type default) (color 0 0 0 0))
   )
-  (wire (pts (xy 113.03 81.28) (xy 111.76 81.28))
+  (wire (pts (xy 130.175 83.82) (xy 128.905 83.82))
+    (stroke (width 0) (type default) (color 0 0 0 0))
+  )
+  (wire (pts (xy 124.46 71.755) (xy 130.175 71.755))
     (stroke (width 0) (type default) (color 0 0 0 0))
   )
@@
     (stroke (width 0) (type default) (color 0 0 0 0))
   )
+  (wire (pts (xy 113.03 71.755) (xy 116.84 71.755))
+    (stroke (width 0) (type default) (color 0 0 0 0))
+  )
   (wire (pts (xy 125.095 59.69) (xy 125.095 66.675))
     (stroke (width 0) (type default) (color 0 0 0 0))
@@
     (effects (font (size 1.27 1.27)) (justify left bottom))
   )
-  (label "AUX_POWER_DETECT" (at 133.35 81.28 180)
+  (label "AUX_POWER_DETECT" (at 150.495 83.82 180)
     (effects (font (size 1.27 1.27)) (justify right bottom))
   )
@@
       (effects (font (size 1.27 1.27)) (justify left))
     )
-    (property "Footprint" "Capacitor_SMD:C_0805_2012Metric" (id 2) (at 65.1002 47.625 0)
+    (property "Footprint" "Capacitor_Tantalum_SMD:CP_EIA-1608-08_AVX-J" (id 2) (at 65.1002 47.625 0)
       (effects (font (size 1.27 1.27)) hide)
     )
@@
     (pin "2")
   )
-  (symbol (lib_id "Device:D_Schottky") (at 127 71.755 0) (unit 1)
+  (symbol (lib_id "Device:D_Schottky") (at 120.65 71.755 0) (unit 1)
     (in_bom yes) (on_board yes)
-    (property "Reference" "D2" (id 0) (at 127 77.2668 0))
-    (property "Value" "D_Schottky" (id 1) (at 127 74.9554 0))
-    (property "Footprint" "Diode_SMD:D_SMA" (id 2) (at 127 71.755 0)
+    (property "Reference" "D2" (id 0) (at 120.65 77.2668 0))
+    (property "Value" "D_Schottky" (id 1) (at 120.65 74.9554 0))
+    (property "Footprint" "Diode_SMD:D_SMA" (id 2) (at 120.65 71.755 0)
       (effects (font (size 1.27 1.27)) hide)
     )
-    (property "Datasheet" "~" (id 3) (at 127 71.755 0)
+    (property "Datasheet" "~" (id 3) (at 120.65 71.755 0)
       (effects (font (size 1.27 1.27)) hide)
     )
-    (property "LCSC" "C22452" (id 4) (at 127 71.755 0)
+    (property "LCSC" "C22452" (id 4) (at 120.65 71.755 0)
       (effects (font (size 1.27 1.27)) hide)
     )
@@
     (pin "1")
   )
-  (symbol (lib_id "Device:R") (at 107.95 81.28 270) (unit 1)
+  (symbol (lib_id "Device:R") (at 125.095 83.82 270) (unit 1)
     (in_bom yes) (on_board yes)
-    (property "Reference" "R14" (id 0) (at 106.68 78.74 90)
+    (property "Reference" "R14" (id 0) (at 123.825 81.28 90)
       (effects (font (size 1.27 1.27)) (justify left))
     )
-    (property "Value" "3.3k" (id 1) (at 106.045 81.28 90)
+    (property "Value" "3.3k" (id 1) (at 123.19 83.82 90)
       (effects (font (size 1.27 1.27)) (justify left))
     )
-    (property "Footprint" "Resistor_SMD:R_0603_1608Metric" (id 2) (at 107.95 79.502 90)
+    (property "Footprint" "Resistor_SMD:R_0603_1608Metric" (id 2) (at 125.095 82.042 90)
       (effects (font (size 1.27 1.27)) hide)
     )
-    (property "Datasheet" "~" (id 3) (at 107.95 81.28 0)
+    (property "Datasheet" "~" (id 3) (at 125.095 83.82 0)
       (effects (font (size 1.27 1.27)) hide)
     )
@@
     (pin "2")
   )
-  (symbol (lib_id "power:GND") (at 102.235 81.28 270) (unit 1)
+  (symbol (lib_id "power:GND") (at 119.38 83.82 270) (unit 1)
     (in_bom yes) (on_board yes)
-    (property "Reference" "#PWR024" (id 0) (at 95.885 81.28 0)
+    (property "Reference" "#PWR024" (id 0) (at 113.03 83.82 0)
       (effects (font (size 1.27 1.27)) hide)
     )
-    (property "Value" "GND" (id 1) (at 97.8408 81.407 0))
-    (property "Footprint" "" (id 2) (at 102.235 81.28 0)
+    (property "Value" "GND" (id 1) (at 114.9858 83.947 0))
+    (property "Footprint" "" (id 2) (at 119.38 83.82 0)
       (effects (font (size 1.27 1.27)) hide)
     )
-    (property "Datasheet" "" (id 3) (at 102.235 81.28 0)
+    (property "Datasheet" "" (id 3) (at 119.38 83.82 0)
       (effects (font (size 1.27 1.27)) hide)
     )
@@
     (pin "2")
   )
-  (symbol (lib_id "Device:R") (at 113.03 75.565 0) (unit 1)
+  (symbol (lib_id "Device:R") (at 130.175 78.105 0) (unit 1)
     (in_bom yes) (on_board yes)
-    (property "Reference" "R12" (id 0) (at 110.49 76.835 90)
+    (property "Reference" "R12" (id 0) (at 127.635 79.375 90)
       (effects (font (size 1.27 1.27)) (justify left))
     )
-    (property "Value" "1.7k" (id 1) (at 113.03 77.47 90)
+    (property "Value" "1.7k" (id 1) (at 130.175 80.01 90)
       (effects (font (size 1.27 1.27)) (justify left))
     )
-    (property "Footprint" "Resistor_SMD:R_0603_1608Metric" (id 2) (at 111.252 75.565 90)
+    (property "Footprint" "Resistor_SMD:R_0603_1608Metric" (id 2) (at 128.397 78.105 90)
       (effects (font (size 1.27 1.27)) hide)
     )
-    (property "Datasheet" "~" (id 3) (at 113.03 75.565 0)
+    (property "Datasheet" "~" (id 3) (at 130.175 78.105 0)
       (effects (font (size 1.27 1.27)) hide)
     )
@@
       (effects (font (size 1.27 1.27)) (justify left))
     )
-    (property "Footprint" "Capacitor_SMD:C_0805_2012Metric" (id 2) (at 93.0402 47.625 0)
+    (property "Footprint" "Capacitor_Tantalum_SMD:CP_EIA-1608-08_AVX-J" (id 2) (at 93.0402 47.625 0)
       (effects (font (size 1.27 1.27)) hide)
     )
@@
     )
     (path "/033fa323-ea5a-4980-be2a-ace9c0c90d5a"
-      (reference "C13") (unit 1) (value "22u") (footprint "Capacitor_SMD:C_0805_2012Metric")
+      (reference "C13") (unit 1) (value "22u") (footprint "Capacitor_Tantalum_SMD:CP_EIA-1608-08_AVX-J")
     )
     (path "/c33635c8-03ae-43d7-81e8-d49b9b5baba3"
-      (reference "C14") (unit 1) (value "22u") (footprint "Capacitor_SMD:C_0805_2012Metric")
+      (reference "C14") (unit 1) (value "22u") (footprint "Capacitor_Tantalum_SMD:CP_EIA-1608-08_AVX-J")
     )
     (path "/ee2973d5-7260-4c80-be23-026eac9d286d"
